File: pidcontroller/powerboard-no-gnd-plane.sch (EAGLE design)
At the start: 41 parts

Commit message: updated eagle files
Parts:
- removed PAD1, PAD10, PAD11, PAD12, PAD13, PAD14, PAD15, PAD16, PAD17, PAD18, PAD19, PAD2, PAD20, PAD21, PAD22, PAD23, PAD24, PAD25, PAD3, PAD4, PAD5, PAD6, PAD7, PAD8, PAD9: (no value), wirepad:2,15/1,0
Changed lines of the file:
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@@
 <part name="GND2" library="supply1" deviceset="GND" device=""/>
 <part name="GND3" library="supply1" deviceset="GND" device=""/>
-<part name="PAD1" library="wirepad" deviceset="2,15/1,0" device=""/>
-<part name="PAD2" library="wirepad" deviceset="2,15/1,0" device=""/>
-<part name="PAD3" library="wirepad" deviceset="2,15/1,0" device=""/>
-<part name="PAD4" library="wirepad" deviceset="2,15/1,0" device=""/>
-<part name="PAD5" library="wirepad" deviceset="2,15/1,0" device=""/>
-<part name="PAD6" library="wirepad" deviceset="2,15/1,0" device=""/>
-<part name="PAD7" library="wirepad" deviceset="2,15/1,0" device=""/>
-<part name="PAD8" library="wirepad" deviceset="2,15/1,0" device=""/>
-<part name="PAD9" library="wirepad" deviceset="2,15/1,0" device=""/>
-<part name="PAD10" library="wirepad" deviceset="2,15/1,0" device=""/>
-<part name="PAD11" library="wirepad" deviceset="2,15/1,0" device=""/>
-<part name="PAD12" library="wirepad" deviceset="2,15/1,0" device=""/>
-<part name="PAD13" library="wirepad" deviceset="2,15/1,0" device=""/>
-<part name="PAD14" library="wirepad" deviceset="2,15/1,0" device=""/>
-<part name="PAD15" library="wirepad" deviceset="2,15/1,0" device=""/>
-<part name="PAD16" library="wirepad" deviceset="2,15/1,0" device=""/>
-<part name="PAD17" library="wirepad" deviceset="2,15/1,0" device=""/>
-<part name="PAD18" library="wirepad" deviceset="2,15/1,0" device=""/>
-<part name="PAD19" library="wirepad" deviceset="2,15/1,0" device=""/>
-<part name="PAD20" library="wirepad" deviceset="2,15/1,0" device=""/>
-<part name="PAD21" library="wirepad" deviceset="2,15/1,0" device=""/>
-<part name="PAD22" library="wirepad" deviceset="2,15/1,0" device=""/>
 <part name="R1" library="pot" deviceset="TRIM_EU-" device="LI10"/>
-<part name="PAD23" library="wirepad" deviceset="2,15/1,0" device=""/>
-<part name="PAD24" library="wirepad" deviceset="2,15/1,0" device=""/>
-<part name="PAD25" library="wirepad" deviceset="2,15/1,0" device=""/>
 </parts>
 <sheets>
@@
 <instance part="GND2" gate="1" x="83.82" y="55.88"/>
 <instance part="GND3" gate="1" x="68.58" y="48.26" rot="R180"/>
-<instance part="PAD1" gate="1" x="66.04" y="81.28"/>
-<instance part="PAD2" gate="1" x="81.28" y="81.28"/>
-<instance part="PAD3" gate="1" x="58.42" y="86.36"/>
-<instance part="PAD4" gate="1" x="53.34" y="81.28"/>
-<instance part="PAD5" gate="1" x="43.18" y="78.74"/>
-<instance part="PAD6" gate="1" x="101.6" y="83.82"/>
-<instance part="PAD7" gate="1" x="104.14" y="78.74"/>
-<instance part="PAD8" gate="1" x="121.92" y="86.36"/>
-<instance part="PAD9" gate="1" x="127" y="81.28"/>
-<instance part="PAD10" gate="1" x="124.46" y="71.12"/>
-<instance part="PAD11" gate="1" x="30.48" y="68.58"/>
-<instance part="PAD12" gate="1" x="33.02" y="78.74"/>
-<instance part="PAD13" gate="1" x="35.56" y="86.36"/>
-<instance part="PAD14" gate="1" x="68.58" y="88.9"/>
-<instance part="PAD15" gate="1" x="86.36" y="88.9"/>
-<instance part="PAD16" gate="1" x="116.84" y="73.66"/>
-<instance part="PAD17" gate="1" x="124.46" y="63.5"/>
-<instance part="PAD18" gate="1" x="124.46" y="55.88"/>
-<instance part="PAD19" gate="1" x="124.46" y="48.26"/>
-<instance part="PAD20" gate="1" x="127" y="40.64"/>
-<instance part="PAD21" gate="1" x="121.92" y="27.94"/>
-<instance part="PAD22" gate="1" x="121.92" y="20.32"/>
 <instance part="R1" gate="1" x="60.96" y="53.34" rot="R270"/>
-<instance part="PAD23" gate="1" x="25.4" y="68.58"/>
-<instance part="PAD24" gate="1" x="25.4" y="73.66"/>
-<instance part="PAD25" gate="1" x="25.4" y="78.74"/>
 </instances>
 <busses>
