File: pidcontroller/powerboard.brd (EAGLE design)
At the start: 68.2 x 45.7 mm, 41 parts

Commit message: updated eagle files
Parts:
- removed PAD1, PAD10, PAD11, PAD12, PAD13, PAD14, PAD15, PAD16, PAD17, PAD18, PAD19, PAD2, PAD20, PAD21, PAD22, PAD23, PAD24, PAD25, PAD3, PAD4, PAD5, PAD6, PAD7, PAD8, PAD9: (no value), wirepad:2,15/1,0
Changed lines of the file:
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@@
 <element name="D6" library="wirepad" package="2,54/1,1" value="" x="38.1" y="20.32"/>
 <element name="D7" library="wirepad" package="2,54/1,1" value="" x="22.86" y="20.32"/>
-<element name="PAD1" library="wirepad" package="2,15/1,0" value="" x="29.21" y="27.94"/>
-<element name="PAD2" library="wirepad" package="2,15/1,0" value="" x="29.21" y="30.48"/>
-<element name="PAD3" library="wirepad" package="2,15/1,0" value="" x="29.21" y="33.02"/>
-<element name="PAD4" library="wirepad" package="2,15/1,0" value="" x="31.75" y="33.02"/>
-<element name="PAD5" library="wirepad" package="2,15/1,0" value="" x="31.75" y="30.48"/>
-<element name="PAD6" library="wirepad" package="2,15/1,0" value="" x="31.75" y="27.94"/>
-<element name="PAD7" library="wirepad" package="2,15/1,0" value="" x="29.21" y="19.05"/>
-<element name="PAD8" library="wirepad" package="2,15/1,0" value="" x="31.75" y="19.05"/>
-<element name="PAD9" library="wirepad" package="2,15/1,0" value="" x="29.21" y="16.51"/>
-<element name="PAD10" library="wirepad" package="2,15/1,0" value="" x="31.75" y="16.51"/>
-<element name="PAD11" library="wirepad" package="2,15/1,0" value="" x="29.21" y="21.59"/>
-<element name="PAD12" library="wirepad" package="2,15/1,0" value="" x="31.75" y="21.59"/>
-<element name="PAD13" library="wirepad" package="2,15/1,0" value="" x="29.21" y="13.97"/>
-<element name="PAD14" library="wirepad" package="2,15/1,0" value="" x="31.75" y="13.97"/>
-<element name="PAD15" library="wirepad" package="2,15/1,0" value="" x="29.21" y="11.43"/>
-<element name="PAD16" library="wirepad" package="2,15/1,0" value="" x="31.75" y="11.43"/>
-<element name="PAD17" library="wirepad" package="2,15/1,0" value="" x="29.21" y="8.89"/>
-<element name="PAD18" library="wirepad" package="2,15/1,0" value="" x="31.75" y="8.89"/>
-<element name="PAD19" library="wirepad" package="2,15/1,0" value="" x="29.21" y="6.35"/>
-<element name="PAD20" library="wirepad" package="2,15/1,0" value="" x="31.75" y="6.35"/>
-<element name="PAD21" library="wirepad" package="2,15/1,0" value="" x="29.21" y="3.81"/>
-<element name="PAD22" library="wirepad" package="2,15/1,0" value="" x="31.75" y="3.81"/>
 <element name="R1" library="pot" package="LI10" value="" x="49.53" y="8.89"/>
-<element name="PAD23" library="wirepad" package="2,15/1,0" value="" x="49.53" y="13.97"/>
-<element name="PAD24" library="wirepad" package="2,15/1,0" value="" x="46.99" y="3.81"/>
-<element name="PAD25" library="wirepad" package="2,15/1,0" value="" x="52.07" y="3.81"/>
 </elements>
 <signals>
