File: pidcontroller/pidcontroller-mega32.brd (EAGLE design)
At the start: 100 x 75.4 mm, 31 parts, among them IC2 MAX3232CWE, IC3 MEGA32-A

Commit message: more changes
Routing:
- net VCC: track 298.6 -> 303.0 mm
- net RESET: track 45.9 -> 49.2 mm
- net 232RX: track 42.0 -> 44.7 mm
- net N$1: track 29.9 -> 32.2 mm
- net N$11: track 10.2 -> 12.2 mm
- net 232TX: track 46.5 -> 48.4 mm
- net N$8: track 9.76 -> 11.2 mm
- net N$7: track 9.65 -> 10.9 mm
- net N$15: track 27.7 -> 28.8 mm
- net N$5: track 9.46 -> 10.4 mm
