File: Raspberry can interface/RPiCanInterface.sch (EAGLE design)
At the start: 16 parts, among them IC1 MCP2515-E/P

Commit message: fixed error on pican board
Connections:
- removed net 3.3V: R3.2, R4.2
- net VCC: now also R3.2, R4.2
Changed lines of the file:
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@@
 <setting verticaltext="up"/>
 </settings>
-<grid distance="0.1" unitdist="inch" unit="inch" style="lines" multiple="1" display="yes" altdistance="0.01" altunitdist="inch" altunit="inch"/>
+<grid distance="0.1" unitdist="inch" unit="inch" style="lines" multiple="1" display="no" altdistance="0.01" altunitdist="inch" altunit="inch"/>
 <layers>
 <layer number="1" name="Top" color="4" fill="1" visible="no" active="no"/>
@@
 </segment>
 </net>
-<net name="3.3V" class="0">
+<net name="VCC" class="0">
+<segment>
+<pinref part="+3V3" gate="P" pin="P"/>
+<pinref part="AFADSF1" gate="VCC" pin="VCC"/>
+<wire x1="5.08" y1="81.28" x2="5.08" y2="86.36" width="0.1524" layer="91"/>
+</segment>
+<segment>
+<pinref part="IC1" gate="G$1" pin="VDD"/>
+<pinref part="P+1" gate="VCC" pin="VCC"/>
+<wire x1="58.42" y1="71.12" x2="58.42" y2="81.28" width="0.1524" layer="91"/>
+</segment>
+<segment>
+<pinref part="R5" gate="G$1" pin="2"/>
+<pinref part="AFADSF2" gate="VCC" pin="VCC"/>
+<wire x1="12.7" y1="83.82" x2="12.7" y2="86.36" width="0.1524" layer="91"/>
+</segment>
 <segment>
 <pinref part="R4" gate="G$1" pin="2"/>
@@
 </segment>
 </net>
-<net name="VCC" class="0">
-<segment>
-<pinref part="+3V3" gate="P" pin="P"/>
-<pinref part="AFADSF1" gate="VCC" pin="VCC"/>
-<wire x1="5.08" y1="81.28" x2="5.08" y2="86.36" width="0.1524" layer="91"/>
-</segment>
-<segment>
-<pinref part="IC1" gate="G$1" pin="VDD"/>
-<pinref part="P+1" gate="VCC" pin="VCC"/>
-<wire x1="58.42" y1="71.12" x2="58.42" y2="81.28" width="0.1524" layer="91"/>
-</segment>
-<segment>
-<pinref part="R5" gate="G$1" pin="2"/>
-<pinref part="AFADSF2" gate="VCC" pin="VCC"/>
-<wire x1="12.7" y1="83.82" x2="12.7" y2="86.36" width="0.1524" layer="91"/>
-</segment>
-</net>
